Commit message: Barrett can barely pick banana

File: assets/fetch/fetch_barretthand.urdf (robot description, URDF)
Before this commit: robot fetch, 38 links, 37 joints
Links:
- added link virtual_grasp_frame, mass 0.0001
Joints:
- added joint virtual_grasp_joint: type fixed, parent bh_base_link, child virtual_grasp_frame, origin xyz=0 0 0 rpy=0 -1.5708 0
